File: robotika.kicad_pcb (KiCad board)
At the start: 2 copper layers, 70 x 50 mm, 0 parts

Commit message: A LOT OF WORK DONE
Added a version using WeMos D1 Mini
Parts:
- added C1: 10u, Capacitor_THT:CP_Radial_D5.0mm_P2.50mm, F.Cu at (109.0, 110.5)
- added C10: 100u, Capacitor_THT:CP_Radial_D5.0mm_P2.50mm, F.Cu at (123.0, 75.0)
- added C2: 100n, Capacitor_SMD:C_0805_2012Metric_Pad1.18x1.45mm_HandSolder, F.Cu at (103.0, 110.0)
- added C3: 1u, Capacitor_SMD:C_0805_2012Metric_Pad1.18x1.45mm_HandSolder, F.Cu at (109.0, 93.5)
- added C4: 100n, Capacitor_SMD:C_0805_2012Metric_Pad1.18x1.45mm_HandSolder, F.Cu at (112.5, 93.5)
- added C5: 10u, Capacitor_THT:CP_Radial_D5.0mm_P2.50mm, F.Cu at (144.0, 90.2)
- added C6: 1u, Capacitor_SMD:C_0805_2012Metric_Pad1.18x1.45mm_HandSolder, F.Cu at (135.0, 89.0)
- added C7: 100n, Capacitor_SMD:C_0805_2012Metric_Pad1.18x1.45mm_HandSolder, F.Cu at (138.5, 89.0)
- added C8: 100n, Capacitor_SMD:C_0805_2012Metric_Pad1.18x1.45mm_HandSolder, F.Cu at (125.0, 90.0)
- added C9: 10u, Capacitor_THT:CP_Radial_D5.0mm_P2.50mm, F.Cu at (104.2, 82.2)
- added H1: MountingHole, MountingHole:MountingHole_3.2mm_M3, F.Cu at (166.5, 116.5)
- added H2: MountingHole, MountingHole:MountingHole_3.2mm_M3, F.Cu at (166.5, 73.5)
- added H3: MountingHole, MountingHole:MountingHole_3.2mm_M3, F.Cu at (103.5, 116.5)
- added H4: MountingHole, MountingHole:MountingHole_3.2mm_M3, F.Cu at (103.5, 73.5)
- added J1: USB_C_Receptacle_USB2.0_16P, Connector_USB:USB_C_Receptacle_XKB_U262-16XN-4BVC11, F.Cu at (115.9, 117.5)
- added J2: 9v BATTERY, Connector_PinHeader_2.54mm:PinHeader_1x02_P2.54mm_Vertical, F.Cu at (140.7, 72.5)
- added J3: MOTOR1, Connector_PinHeader_2.54mm:PinHeader_1x02_P2.54mm_Vertical, F.Cu at (166.5, 107.0)
- added J4: MOTOR2, Connector_PinHeader_2.54mm:PinHeader_1x02_P2.54mm_Vertical, F.Cu at (166.5, 80.5)
- added R1: 5.1k, Resistor_SMD:R_0805_2012Metric_Pad1.20x1.40mm_HandSolder, F.Cu at (118.6, 110.5)
- added R2: 5.1k, Resistor_SMD:R_0805_2012Metric_Pad1.20x1.40mm_HandSolder, F.Cu at (113.3, 110.5)
- added R3: 10k, Resistor_SMD:R_0805_2012Metric_Pad1.20x1.40mm_HandSolder, F.Cu at (146.6, 108.0)
- added SW1: RESET, Button_Switch_THT:SW_PUSH_6mm, F.Cu at (148.2, 112.2)
- added SW2: power, Connector_PinSocket_2.54mm:PinSocket_1x03_P2.54mm_Vertical, F.Cu at (130.4, 72.4)
- added U1: AMS1117-3.3, Package_TO_SOT_SMD:SOT-223-3_TabPin2, F.Cu at (106.5, 101.5)
- added U2: CH340C, Package_SO:SOIC-16_3.9x9.9mm_P1.27mm, F.Cu at (118.5, 98.8)
- added U3: ESP-12F, RF_Module:ESP-12E, F.Cu at (135.0, 107.5)
- added U4: AMS1117-3.3, Package_TO_SOT_SMD:SOT-223-3_TabPin2, F.Cu at (126.1, 83.5)
- added U5: L7805, Package_TO_SOT_SMD:TO-263-2, F.Cu at (114.5, 77.8)
- added U6: L293D, Package_DIP:DIP-16_W7.62mm, F.Cu at (153.9, 84.3)
Routing:
- net +3.3V: track 0.00 -> 105.9 mm, vias 0 -> 2
- net +5V: track 0.00 -> 96.7 mm, vias 0 -> 1
- net +9V: track 0.00 -> 80.4 mm, vias 0 -> 1
- net 4A: track 0.00 -> 42.4 mm, vias 0 -> 1
- net 3A: track 0.00 -> 32.5 mm, vias 0 -> 2
- net Net-(J3-Pin_1): track 0.00 -> 26.7 mm
- net 1A: track 0.00 -> 26.5 mm
- net Net-(J3-Pin_2): track 0.00 -> 25.7 mm
- net RX: track 0.00 -> 23.6 mm, vias 0 -> 2
- net Net-(J4-Pin_1): track 0.00 -> 22.0 mm
- net TX: track 0.00 -> 20.2 mm
- net D+: track 0.00 -> 20.0 mm, vias 0 -> 2
- net VBUS: track 0.00 -> 19.9 mm
- net Net-(U3-~{RST}): track 0.00 -> 18.6 mm
- net D-: track 0.00 -> 18.3 mm
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- added copper zone on B.Cu, net GND
- added copper zone on F.Cu, net GND
