File: robotika.kicad_sch (KiCad schematic)
At the start: 25 parts, among them J1 9v BATTERY, J2 USB_C_Receptacle_USB2.0_16P, J3 MOTOR1, J4 MOTOR2, SW1 POWER, SW2 SW_Push, U1 ESP-12F, U2 CH340C, U3 L293D, U4 AMS1117-3.3, U6 L7805, U7 AMS1117-3.3

Commit message: Schematic Update 2
Parts:
- removed C1, C10, C2, C4: 10u, symbol Device:C
- added C10: 100u, symbol Device:C_Polarized
- added C3, C5, C9: 10u, symbol Device:C_Polarized
- J2: renamed from J1; footprint (none) -> Connector_PinHeader_2.54mm:PinHeader_1x02_P2.54mm_Vertical
- J3, J4: footprint (none) -> Connector_PinHeader_2.54mm:PinHeader_1x02_P2.54mm_Vertical
- R1, R2, R3: footprint (none) -> Resistor_SMD:R_0805_2012Metric_Pad1.20x1.40mm_HandSolder
- SW1: renamed from SW2; footprint (none) -> Button_Switch_THT:SW_PUSH_6mm
- renumbered C6 to C1, C7 to C2, C5 to C4, C3 to C6, C8 to C7, C9 to C8, J2 to J1, SW1 to SW2, U7 to U1, U1 to U3, U6 to U5, U3 to U6
Connections:
- net +3.3V: now also C5.1
- net +5V: now also C9.1
- net +9V: now also C10.1
- net GND: now also C10.2, C3.2, C5.2, C9.2
- net VBUS: now also C3.1

Commit message: A LOT OF WORK DONE
Added a version using WeMos D1 Mini
Parts:
- removed C6: 100n, symbol Device:C
- removed SW2: POWER, symbol Switch:SW_SPST
- added C8: 100n, Capacitor_SMD:C_0805_2012Metric_Pad1.18x1.45mm_HandSolder, symbol Device:C
- added H1, H2, H3, H4: MountingHole, MountingHole:MountingHole_3.2mm_M3, symbol Mechanical:MountingHole
- added SW2: power, Connector_PinSocket_2.54mm:PinSocket_1x03_P2.54mm_Vertical, symbol Switch:SW_SPDT
- C1: renamed from C3; footprint (none) -> Capacitor_THT:CP_Radial_D5.0mm_P2.50mm
- C10, C5, C9: footprint (none) -> Capacitor_THT:CP_Radial_D5.0mm_P2.50mm
- C2: renamed from C4; footprint (none) -> Capacitor_SMD:C_0805_2012Metric_Pad1.18x1.45mm_HandSolder
- C3: renamed from C1; value 10u -> 1u; footprint (none) -> Capacitor_SMD:C_0805_2012Metric_Pad1.18x1.45mm_HandSolder
- C4: renamed from C2; footprint (none) -> Capacitor_SMD:C_0805_2012Metric_Pad1.18x1.45mm_HandSolder
- C6: renamed from C7; footprint (none) -> Capacitor_SMD:C_0805_2012Metric_Pad1.18x1.45mm_HandSolder
- C7: renamed from C8; footprint (none) -> Capacitor_SMD:C_0805_2012Metric_Pad1.18x1.45mm_HandSolder
- J1: footprint (none) -> Connector_USB:USB_C_Receptacle_XKB_U262-16XN-4BVC11
- SW1: value SW_Push -> RESET
Connections:
- net +3.3V: now also C8.1
- net +9V: now also SW2.2 (B)
- net GND: now also C8.2
- net at U3.19 (GPIO4): no longer U6.2 (1A)
- net at U3.20 (GPIO5): no longer U6.7 (2A)
- net 1A: now reaches U3.4 (GPIO16)
- net 1A: now also U6.2 (1A)
- net 2A: now reaches U3.5 (GPIO14)
- net 2A: now also U6.7 (2A)
- net 3A: now reaches U3.6 (GPIO12), U6.10 (3A)
- net 4A: now reaches U3.7 (GPIO13), U6.15 (4A)
- net at J2.1 (Pin_1): now also SW2.3 (C)
- no-connect marks 22 -> 23
Other:
- moved on the sheet: C3, C4, C5, C6, C7, R3, SW1, U2, U3
