File: WEMOS VER/wemos/wemos.kicad_sch (KiCad schematic)
At the start: 15 parts, among them J1 9V BATT, J2 MOTOR 1, J3 MOTOR 2, SW1 RESET, SW2 ON/OFF, U1 WeMos D1 Mini, U2 L7805, U3 L293D

Commit message: A LOT OF WORK
Parts:
- added C3: 100n, Capacitor_THT:C_Disc_D5.0mm_W2.5mm_P5.00mm, symbol Device:C
- added C4: 100u, Capacitor_THT:CP_Radial_D5.0mm_P2.50mm, symbol Device:C_Polarized
- added H5, H6, H7, H8: MountingHole, MountingHole:MountingHole_3.2mm_M3, symbol Mechanical:MountingHole
- added J4: 9V BATT, Connector_PinHeader_2.54mm:PinHeader_1x02_P2.54mm_Vertical, symbol Connector:Conn_01x02_Socket
- added J5: MOTOR 1, Connector_PinHeader_2.54mm:PinHeader_1x02_P2.54mm_Vertical, symbol Connector:Conn_01x02_Socket
- added J6: MOTOR 2, Connector_PinHeader_2.54mm:PinHeader_1x02_P2.54mm_Vertical, symbol Connector:Conn_01x02_Socket
- added J7: Conn_01x04_Pin, Connector_PinSocket_2.54mm:PinSocket_1x04_P2.54mm_Vertical, symbol Connector:Conn_01x04_Pin
- added R2: 10k, Resistor_THT:R_Axial_DIN0207_L6.3mm_D2.5mm_P7.62mm_Horizontal, symbol Device:R
- added SW3: RESET, Button_Switch_THT:SW_PUSH_6mm, symbol Switch:SW_Push
- added SW4: ON/OFF, Connector_PinSocket_2.54mm:PinSocket_1x03_P2.54mm_Vertical, symbol Switch:SW_SPDT
- added U4: WeMos D1 Mini, Module:WEMOS_D1_mini_light, symbol MCU_Module:WeMos_D1_mini
- added U5: L7805, Package_TO_SOT_THT:TO-220-3_Vertical, symbol Regulator_Linear:L7805
- added U6: L293D, Package_DIP:DIP-16_W7.62mm, symbol Driver_Motor:L293D
- C1: footprint Capacitor_SMD:C_0805_2012Metric_Pad1.18x1.45mm_HandSolder -> Capacitor_THT:C_Disc_D5.0mm_W2.5mm_P5.00mm
- R1: footprint Resistor_SMD:R_0805_2012Metric_Pad1.20x1.40mm_HandSolder -> Resistor_THT:R_Axial_DIN0207_L6.3mm_D2.5mm_P7.62mm_Horizontal
- U2: footprint Package_TO_SOT_SMD:TO-263-2 -> Package_TO_SOT_THT:TO-220-3_Vertical
Connections:
- net +5V: now also U3.1 (EN1,2), U3.9 (EN3,4)
- net at U1.11 (D4): now also U3.15 (4A); no longer U3.9 (EN3,4)
- net at U1.12 (D3): now also U3.10 (3A); no longer U3.1 (EN1,2)
- net at U1.4 (SCK/D5): no longer U3.10 (3A)
- net at U1.5 (MISO/D6): no longer U3.15 (4A)
- new net: J5.1 (Pin_1), U6.3 (1Y)
- new net: J5.2 (Pin_2), U6.6 (2Y)
- new net: U4.12 (D3), U6.10 (3A)
- new net: J6.1 (Pin_1), U6.11 (3Y)
- new net: J6.2 (Pin_2), U6.14 (4Y)
- new net: U4.11 (D4), U6.15 (4A)
- new net: U4.14 (SCL/D1), U6.2 (1A)
- new net: U4.13 (SDA/D2), U6.7 (2A)
- new net: R2.2, SW3.2, U4.1 (~{RST})
- new net: J7.4 (Pin_4), U4.4 (SCK/D5)
- new net: J7.3 (Pin_3), U4.5 (MISO/D6)
- new net: J7.2 (Pin_2), U4.6 (MOSI/D7)
- new net: J7.1 (Pin_1), U4.7 (CS/D8)
- new net: R2.1, U4.8 (3V3)
- new net: J4.1 (Pin_1), SW4.3 (C)
- new net +5VA: C3.1, U4.9 (5V), U5.1 (IN), U6.1 (EN1,2), U6.16 (VCC1), U6.9 (EN3,4)
- new net +9VA: C4.1, SW4.2 (B), U5.3 (OUT), U6.8 (VCC2)
- new net GND1: C3.2, C4.2, J4.2 (Pin_2), SW3.1, U4.10 (GND), U5.2 (GND), U6.12 (GND), U6.13 (GND), U6.4 (GND), U6.5 (GND)
- no-connect marks 7 -> 14

Commit message: work
Connections:
- net +5V: now also U2.3 (OUT); no longer U2.1 (IN)
- net +5VA: now also U5.3 (OUT); no longer U5.1 (IN)
- net +9V: now also U2.1 (IN); no longer U2.3 (OUT)
- net +9VA: now also U5.1 (IN); no longer U5.3 (OUT)
Changed lines of the file:
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@@
 	)
 	(junction
-		(at 364.49 109.22)
+		(at 105.41 106.68)
 		(diameter 0)
 		(color 0 0 0 0)
 	)
 	(junction
-		(at 96.52 115.57)
+		(at 350.52 100.33)
 		(diameter 0)
 		(color 0 0 0 0)
 	)
 	(junction
-		(at 105.41 106.68)
+		(at 111.76 106.68)
 		(diameter 0)
 		(color 0 0 0 0)
 	)
 	(junction
-		(at 111.76 106.68)
+		(at 364.49 109.22)
 		(diameter 0)
 		(color 0 0 0 0)
@@
 	)
 	(junction
-		(at 82.55 106.68)
+		(at 441.96 83.82)
 		(diameter 0)
 		(color 0 0 0 0)
 	)
 	(junction
-		(at 441.96 83.82)
+		(at 378.46 100.33)
 		(diameter 0)
 		(color 0 0 0 0)
 	)
 	(junction
-		(at 350.52 100.33)
+		(at 105.41 115.57)
 		(diameter 0)
 		(color 0 0 0 0)
 	)
 	(junction
-		(at 378.46 100.33)
+		(at 96.52 115.57)
 		(diameter 0)
 		(color 0 0 0 0)
 	)
 	(junction
-		(at 105.41 115.57)
+		(at 82.55 106.68)
 		(diameter 0)
 		(color 0 0 0 0)
@@
 	)
 	(junction
-		(at 336.55 46.99)
+		(at 373.38 100.33)
 		(diameter 0)
 		(color 0 0 0 0)
 	)
 	(junction
-		(at 68.58 53.34)
+		(at 336.55 46.99)
 		(diameter 0)
 		(color 0 0 0 0)
 	)
 	(junction
-		(at 373.38 100.33)
+		(at 68.58 53.34)
 		(diameter 0)
 		(color 0 0 0 0)
@@
 	(wire
 		(pts
-			(xy 146.05 60.96) (xy 146.05 68.58)
+			(xy 350.52 100.33) (xy 356.87 100.33)
 		)
 		(stroke
@@
 	(wire
 		(pts
-			(xy 82.55 106.68) (xy 88.9 106.68)
+			(xy 146.05 60.96) (xy 146.05 68.58)
 		)
 		(stroke
@@
 	(wire
 		(pts
+			(xy 364.49 107.95) (xy 364.49 109.22)
+		)
+		(stroke
+			(width 0)
+			(type default)
+		)
+	)
+	(wire
+		(pts
 			(xy 88.9 31.75) (xy 68.58 31.75)
 		)
@@
 	(wire
 		(pts
+			(xy 96.52 114.3) (xy 96.52 115.57)
+		)
+		(stroke
+			(width 0)
+			(type default)
+		)
+	)
+	(wire
+		(pts
 			(xy 336.55 46.99) (xy 344.17 46.99)
 		)
@@
 	(wire
 		(pts
-			(xy 96.52 115.57) (xy 105.41 115.57)
+			(xy 82.55 115.57) (xy 96.52 115.57)
 		)
 		(stroke
@@
 	(wire
 		(pts
+			(xy 82.55 106.68) (xy 88.9 106.68)
+		)
+		(stroke
+			(width 0)
+			(type default)
+		)
+	)
+	(wire
+		(pts
 			(xy 466.09 63.5) (xy 457.2 63.5)
 		)
@@
 	(wire
 		(pts
-			(xy 96.52 55.88) (xy 154.94 55.88)
+			(xy 364.49 109.22) (xy 373.38 109.22)
 		)
 		(stroke
@@
 	(wire
 		(pts
-			(xy 68.58 31.75) (xy 68.58 38.1)
+			(xy 96.52 55.88) (xy 154.94 55.88)
 		)
 		(stroke
@@
 	(wire
 		(pts
-			(xy 373.38 109.22) (xy 392.43 109.22)
+			(xy 68.58 31.75) (xy 68.58 38.1)
 		)
 		(stroke
@@
 	(wire
 		(pts
-			(xy 364.49 49.53) (xy 426.72 49.53)
+			(xy 104.14 106.68) (xy 105.41 106.68)
 		)
 		(stroke
@@
 	(wire
 		(pts
-			(xy 466.09 48.26) (xy 457.2 48.26)
+			(xy 373.38 109.22) (xy 392.43 109.22)
 		)
 		(stroke
@@
 	(wire
 		(pts
-			(xy 154.94 55.88) (xy 154.94 53.34)
+			(xy 364.49 49.53) (xy 426.72 49.53)
 		)
 		(stroke
@@
 	(wire
 		(pts
-			(xy 364.49 59.69) (xy 370.84 59.69)
+			(xy 466.09 48.26) (xy 457.2 48.26)
 		)
 		(stroke
@@
 	(wire
 		(pts
-			(xy 382.27 97.79) (xy 382.27 100.33)
+			(xy 154.94 55.88) (xy 154.94 53.34)
 		)
 		(stroke
@@
 	(wire
 		(pts
-			(xy 82.55 115.57) (xy 96.52 115.57)
+			(xy 364.49 59.69) (xy 370.84 59.69)
 		)
 		(stroke
@@
 	(wire
 		(pts
-			(xy 441.96 82.55) (xy 441.96 83.82)
+			(xy 382.27 97.79) (xy 382.27 100.33)
 		)
 		(stroke
@@
 	(wire
 		(pts
-			(xy 173.99 88.9) (xy 173.99 90.17)
+			(xy 441.96 82.55) (xy 441.96 83.82)
 		)
 		(stroke
@@
 	(wire
 		(pts
-			(xy 373.38 100.33) (xy 378.46 100.33)
+			(xy 173.99 88.9) (xy 173.99 90.17)
 		)
 		(stroke
@@
 	(wire
 		(pts
-			(xy 142.24 73.66) (xy 163.83 73.66)
+			(xy 373.38 100.33) (xy 378.46 100.33)
 		)
 		(stroke
@@
 	(wire
 		(pts
-			(xy 96.52 63.5) (xy 142.24 63.5)
+			(xy 142.24 73.66) (xy 163.83 73.66)
 		)
 		(stroke
@@
 	(wire
 		(pts
-			(xy 457.2 52.07) (xy 457.2 50.8)
+			(xy 96.52 63.5) (xy 142.24 63.5)
 		)
 		(stroke
@@
 	(wire
 		(pts
-			(xy 350.52 100.33) (xy 356.87 100.33)
+			(xy 457.2 52.07) (xy 457.2 50.8)
 		)
 		(stroke
@@
 	(wire
 		(pts
-			(xy 364.49 107.95) (xy 364.49 109.22)
-		)
-		(stroke
-			(width 0)
-			(type default)
-		)
-	)
-	(wire
-		(pts
-			(xy 96.52 114.3) (xy 96.52 115.57)
-		)
-		(stroke
-			(width 0)
-			(type default)
-		)
-	)
-	(wire
-		(pts
 			(xy 350.52 107.95) (xy 350.52 109.22)
 		)
@@
 	(wire
 		(pts
-			(xy 364.49 109.22) (xy 373.38 109.22)
+			(xy 189.23 73.66) (xy 189.23 72.39)
 		)
 		(stroke
@@
 	(wire
 		(pts
-			(xy 189.23 73.66) (xy 189.23 72.39)
+			(xy 68.58 53.34) (xy 76.2 53.34)
 		)
 		(stroke
@@
 	(wire
 		(pts
-			(xy 68.58 53.34) (xy 76.2 53.34)
+			(xy 96.52 115.57) (xy 105.41 115.57)
 		)
 		(stroke
@@
 	(wire
 		(pts
-			(xy 104.14 106.68) (xy 105.41 106.68)
-		)
-		(stroke
-			(width 0)
-			(type default)
-		)
-	)
-	(wire
-		(pts
 			(xy 422.91 62.23) (xy 431.8 62.23)
 		)
@@
 		(lib_id "Regulator_Linear:L7805")
 		(at 96.52 106.68 0)
+		(mirror y)
 		(unit 1)
 		(exclude_from_sim no)
@@
 		(on_board yes)
 		(dnp no)
-		(fields_autoplaced yes)
 		(property "Reference" "U2"
 			(at 96.52 100.33 0)
@@
 		)
 		(property "Footprint" "Package_TO_SOT_THT:TO-220-3_Vertical"
-			(at 97.155 110.49 0)
+			(at 95.885 110.49 0)
 			(effects
 				(font
@@
 		(lib_id "Regulator_Linear:L7805")
 		(at 364.49 100.33 0)
+		(mirror y)
 		(unit 1)
 		(exclude_from_sim no)
@@
 		(on_board yes)
 		(dnp no)
-		(fields_autoplaced yes)
 		(property "Reference" "U5"
 			(at 364.49 93.98 0)
@@
 		)
 		(property "Footprint" "Package_TO_SOT_THT:TO-220-3_Vertical"
-			(at 365.125 104.14 0)
+			(at 363.855 104.14 0)
 			(effects
 				(font

Commit message: slight changes
Parts:
- removed C3: 100n, Capacitor_THT:C_Disc_D5.0mm_W2.5mm_P5.00mm, symbol Device:C
- removed C4: 100u, Capacitor_THT:CP_Radial_D5.0mm_P2.50mm, symbol Device:C_Polarized
- removed H5, H6, H7, H8: MountingHole, MountingHole:MountingHole_3.2mm_M3, symbol Mechanical:MountingHole
- removed J4: 9V BATT, Connector_PinHeader_2.54mm:PinHeader_1x02_P2.54mm_Vertical, symbol Connector:Conn_01x02_Socket
- removed J5: MOTOR 1, Connector_PinHeader_2.54mm:PinHeader_1x02_P2.54mm_Vertical, symbol Connector:Conn_01x02_Socket
- removed J6: MOTOR 2, Connector_PinHeader_2.54mm:PinHeader_1x02_P2.54mm_Vertical, symbol Connector:Conn_01x02_Socket
- removed J7: Conn_01x04_Pin, Connector_PinSocket_2.54mm:PinSocket_1x04_P2.54mm_Vertical, symbol Connector:Conn_01x04_Pin
- removed R2: 10k, Resistor_THT:R_Axial_DIN0207_L6.3mm_D2.5mm_P7.62mm_Horizontal, symbol Device:R
- removed SW3: RESET, Button_Switch_THT:SW_PUSH_6mm, symbol Switch:SW_Push
- removed SW4: ON/OFF, Connector_PinSocket_2.54mm:PinSocket_1x03_P2.54mm_Vertical, symbol Switch:SW_SPDT
- removed U4: WeMos D1 Mini, Module:WEMOS_D1_mini_light, symbol MCU_Module:WeMos_D1_mini
- removed U5: L7805, Package_TO_SOT_THT:TO-220-3_Vertical, symbol Regulator_Linear:L7805
- removed U6: L293D, Package_DIP:DIP-16_W7.62mm, symbol Driver_Motor:L293D
Connections:
- no-connect marks 14 -> 9
