File: WEMOS VER/wemos/wemos.kicad_pcb (KiCad board)
At the start: 2 copper layers, 50 x 50 mm, 15 parts, among them J1 9V BATT, J2 MOTOR 1, J3 MOTOR 2, SW1 RESET, SW2 ON/OFF, U1 WeMos D1 Mini, U2 L7805, U3 L293D

Commit message: A LOT OF WORK
Parts:
- added C3: 100n, Capacitor_THT:C_Disc_D5.0mm_W2.5mm_P5.00mm, F.Cu at (49.5, 48.0)
- added C4: 100u, Capacitor_THT:CP_Radial_D5.0mm_P2.50mm, F.Cu at (80.7, 86.2)
- added H5: MountingHole, MountingHole:MountingHole_3.2mm_M3, F.Cu at (44.5, 41.0)
- added H6: MountingHole, MountingHole:MountingHole_3.2mm_M3, F.Cu at (87.5, 41.0)
- added H7: MountingHole, MountingHole:MountingHole_3.2mm_M3, F.Cu at (44.5, 94.0)
- added H8: MountingHole, MountingHole:MountingHole_3.2mm_M3, F.Cu at (87.5, 94.0)
- added J4: 9V BATT, Connector_PinHeader_2.54mm:PinHeader_1x02_P2.54mm_Vertical, F.Cu at (86.5, 61.0)
- added J5: MOTOR 1, Connector_PinHeader_2.54mm:PinHeader_1x02_P2.54mm_Vertical, F.Cu at (76.5, 93.5)
- added J6: MOTOR 2, Connector_PinHeader_2.54mm:PinHeader_1x02_P2.54mm_Vertical, F.Cu at (52.2, 93.5)
- added J7: Conn_01x04_Pin, Connector_PinSocket_2.54mm:PinSocket_1x04_P2.54mm_Vertical, F.Cu at (86.5, 47.9)
- added R2: 10k, Resistor_THT:R_Axial_DIN0207_L6.3mm_D2.5mm_P7.62mm_Horizontal, F.Cu at (72.5, 56.2)
- added SW3: RESET, Button_Switch_THT:SW_PUSH_6mm, F.Cu at (88.2, 73.2)
- added SW4: ON/OFF, Connector_PinSocket_2.54mm:PinSocket_1x03_P2.54mm_Vertical, F.Cu at (86.0, 81.4)
- added U4: WeMos D1 Mini, Module:WEMOS_D1_mini_light, F.Cu at (77.4, 63.9)
- added U5: L7805, Package_TO_SOT_THT:TO-220-3_Vertical, F.Cu at (46.6, 54.0)
- added U6: L293D, Package_DIP:DIP-16_W7.62mm, F.Cu at (57.1, 88.5)
- C1: footprint Capacitor_SMD:C_0805_2012Metric_Pad1.18x1.45mm_HandSolder -> Capacitor_THT:C_Disc_D5.0mm_W2.5mm_P5.00mm
- R1: footprint Resistor_SMD:R_0805_2012Metric_Pad1.20x1.40mm_HandSolder -> Resistor_THT:R_Axial_DIN0207_L6.3mm_D2.5mm_P7.62mm_Horizontal
- U2: footprint Package_TO_SOT_SMD:TO-263-2 -> Package_TO_SOT_THT:TO-220-3_Vertical
- moved C1 64.0 mm to (120.5, 48.5), turned to 180 degrees
- moved SW1 57.7 mm to (153.5, 58.8), turned to 0 degrees
- moved U2 52.4 mm to (117.0, 55.9), turned to -90 degrees
- moved H1 48.1 mm to (115.5, 40.5)
- moved H2 48.1 mm to (158.5, 40.5)
- moved U3 46.1 mm to (128.3, 85.5)
- moved J1 45.4 mm to (157.0, 51.3), turned to 180 degrees
- moved R1 43.7 mm to (144.0, 55.7), turned to -90 degrees
- moved C2 43.0 mm to (153.0, 83.3), turned to -90 degrees
- moved J2 42.3 mm to (147.7, 92.0), turned to 90 degrees
- moved H3 38.1 mm to (115.5, 93.5)
- moved H4 38.1 mm to (158.5, 93.5)
- moved U1 36.3 mm to (148.4, 63.4), turned to 180 degrees
- moved SW2 35.5 mm to (156.5, 72.5)
- moved J3 21.3 mm to (123.7, 92.0), turned to 90 degrees
Connections:
- U1 pad 4: Net-(U1-SCK/D5) -> unconnected-(U1-SCK/D5-Pad4)
- U1 pad 5: Net-(U1-MISO/D6) -> unconnected-(U1-MISO/D6-Pad5)
- U3 pad 1: Net-(U1-D3) -> +5V
- U3 pad 10: Net-(U1-SCK/D5) -> Net-(U1-D3)
- U3 pad 15: Net-(U1-MISO/D6) -> Net-(U1-D4)
- U3 pad 9: Net-(U1-D4) -> +5V
Routing:
- net +9VA: track 0.00 -> 78.2 mm, vias 0 -> 2
- net +5VA: track 0.00 -> 73.2 mm, vias 0 -> 2
- net Net-(U4-SCL/D1): track 0.00 -> 57.0 mm
- net Net-(U4-SDA/D2): track 0.00 -> 47.3 mm
- net Net-(J6-Pin_1): track 0.00 -> 39.5 mm
- net Net-(U4-D3): track 0.00 -> 37.5 mm, vias 0 -> 2
- net Net-(J4-Pin_1): track 0.00 -> 34.0 mm
- net Net-(U1-SCK/D5): track 33.8 -> 0.00 mm
- net Net-(U4-D4): track 0.00 -> 33.3 mm, vias 0 -> 2
- net +9V: track 53.2 -> 82.5 mm, vias 1 -> 2
- net Net-(J6-Pin_2): track 0.00 -> 28.1 mm
- net +5V: track 44.0 -> 70.3 mm, vias 1 -> 2
- net Net-(U1-MISO/D6): track 21.6 -> 0.00 mm
- net Net-(J5-Pin_1): track 0.00 -> 17.9 mm
- net Net-(J3-Pin_1): track 27.4 -> 45.2 mm, vias 1 -> 0
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- added copper zone on B.Cu, net GND1
- added copper zone on F.Cu, net GND1
Other:
- board size 50 x 50 mm -> 121 x 60.5 mm
- board text added: "+"
- board text added: "-"
- board text added: "CS/SS"
- board text added: "MISO"
- board text added: "MOSI"
- board text added: "SCK"
- board text removed: "OFF"
- board text removed: "ON"

Commit message: work
Parts:
- moved U2 5.08 mm to (116.9, 61.0), turned to 90 degrees
- moved U5 4.58 mm to (46.5, 58.5), turned to 90 degrees
Connections:
- U2 pad 1: +5V -> +9V
- U2 pad 3: +9V -> +5V
- U5 pad 1: +5VA -> +9VA
- U5 pad 3: +9VA -> +5VA

Commit message: slight changes
Parts:
- removed C3: 100n, Capacitor_THT:C_Disc_D5.0mm_W2.5mm_P5.00mm
- removed C4: 100u, Capacitor_THT:CP_Radial_D5.0mm_P2.50mm
- removed H5, H6, H7, H8: MountingHole, MountingHole:MountingHole_3.2mm_M3
- removed J4: 9V BATT, Connector_PinHeader_2.54mm:PinHeader_1x02_P2.54mm_Vertical
- removed J5: MOTOR 1, Connector_PinHeader_2.54mm:PinHeader_1x02_P2.54mm_Vertical
- removed J6: MOTOR 2, Connector_PinHeader_2.54mm:PinHeader_1x02_P2.54mm_Vertical
- removed J7: Conn_01x04_Pin, Connector_PinSocket_2.54mm:PinSocket_1x04_P2.54mm_Vertical
- removed R2: 10k, Resistor_THT:R_Axial_DIN0207_L6.3mm_D2.5mm_P7.62mm_Horizontal
- removed SW3: RESET, Button_Switch_THT:SW_PUSH_6mm
- removed SW4: ON/OFF, Connector_PinSocket_2.54mm:PinSocket_1x03_P2.54mm_Vertical
- removed U4: WeMos D1 Mini, Module:WEMOS_D1_mini_light
- removed U5: L7805, Package_TO_SOT_THT:TO-220-3_Vertical
- removed U6: L293D, Package_DIP:DIP-16_W7.62mm
- moved U3 56.4 mm to (71.9, 87.1)
- moved H1 56.4 mm to (59.1, 42.1)
- moved H3 56.4 mm to (59.1, 95.1)
- moved C1 56.4 mm to (64.1, 50.1)
- moved C2 56.4 mm to (96.6, 84.9)
- moved H2 56.4 mm to (102.1, 42.1)
- moved H4 56.4 mm to (102.1, 95.1)
- moved J1 56.4 mm to (100.6, 52.9)
- moved J2 56.4 mm to (91.3, 93.6)
- moved J3 56.4 mm to (67.3, 93.6)
- moved R1 56.4 mm to (87.6, 57.3)
- moved SW1 56.4 mm to (97.1, 60.4)
- moved SW2 56.4 mm to (100.1, 74.1)
- moved U1 56.4 mm to (92.1, 65.0)
- moved U2 56.4 mm to (60.6, 62.6)
Routing:
- net +9VA: track 78.2 -> 0.00 mm, vias 2 -> 0
- net +5VA: track 72.9 -> 0.00 mm, vias 2 -> 0
- net Net-(U4-SCL/D1): track 57.0 -> 0.00 mm
- net Net-(U4-SDA/D2): track 47.3 -> 0.00 mm
- net Net-(J6-Pin_1): track 39.5 -> 0.00 mm
- net Net-(U4-D3): track 37.5 -> 0.00 mm, vias 2 -> 0
- net Net-(J4-Pin_1): track 34.0 -> 0.00 mm
- net Net-(U4-D4): track 33.3 -> 0.00 mm, vias 2 -> 0
- net Net-(J6-Pin_2): track 28.1 -> 0.00 mm
- net Net-(J5-Pin_1): track 17.9 -> 0.00 mm
- net Net-(U4-3V3): track 14.2 -> 0.00 mm
- net Net-(J5-Pin_2): track 12.9 -> 0.00 mm
- net Net-(U4-~{RST}): track 11.6 -> 0.00 mm
- net Net-(J7-Pin_4): track 9.37 -> 0.00 mm
- net Net-(J7-Pin_3): track 9.37 -> 0.00 mm
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- removed copper zone on B.Cu, net GND1
- removed copper zone on F.Cu, net GND1
Other:
- board size 121 x 60.5 mm -> 50 x 60 mm
- board text removed: "CS/SS"
- board text removed: "MISO"
- board text removed: "MOSI"
- board text removed: "SCK"

Commit message: slight change to pcb
Parts:
- added ?: , , F.Cu at (86.9, 69.8)
- added ?: , , F.Cu at (70.4, 76.5)
- added ?: , , F.Cu at (73.7, 76.7)
- added ?: , , F.Cu at (96.8, 46.0)
- added ?: , , F.Cu at (64.5, 44.2)
- added ?: , , F.Cu at (86.9, 73.4)
- added REF**: SolderWire-0.5sqmm_1x01_D0.9mm_OD2.3mm, Connector_Wire:SolderWire-0.5sqmm_1x01_D0.9mm_OD2.3mm, F.Cu at (62.5, 89.4)
- added REF**: SolderWire-0.5sqmm_1x01_D0.9mm_OD2.3mm, Connector_Wire:SolderWire-0.5sqmm_1x01_D0.9mm_OD2.3mm, F.Cu at (92.7, 88.9)
- added REF**: SolderWire-0.5sqmm_1x01_D0.9mm_OD2.3mm, Connector_Wire:SolderWire-0.5sqmm_1x01_D0.9mm_OD2.3mm, F.Cu at (82.5, 65.5)
- added REF**: SolderWire-0.5sqmm_1x01_D0.9mm_OD2.3mm, Connector_Wire:SolderWire-0.5sqmm_1x01_D0.9mm_OD2.3mm, F.Cu at (65.5, 68.6)
- added REF**: SolderWire-0.5sqmm_1x01_D0.9mm_OD2.3mm, Connector_Wire:SolderWire-0.5sqmm_1x01_D0.9mm_OD2.3mm, F.Cu at (72.9, 52.6)
- added REF**: SolderWire-0.5sqmm_1x01_D0.9mm_OD2.3mm, Connector_Wire:SolderWire-0.5sqmm_1x01_D0.9mm_OD2.3mm, F.Cu at (79.5, 67.3)
Routing:
- net Net-(U1-~{RST}): track 9.59 -> 16.1 mm
- net Net-(J3-Pin_2): track 31.2 -> 34.7 mm
- net Net-(U1-D4): track 30.9 -> 29.0 mm, vias 2 -> 0
- net Net-(U1-SDA/D2): track 48.1 -> 49.9 mm, vias 2 -> 0
- net Net-(U1-SCL/D1): track 57.3 -> 58.2 mm, vias 2 -> 0
- net +9V: vias 2 -> 0
- net +5V: vias 2 -> 0

Commit message: pdf pcb
Parts:
- moved REF** 0.80 mm to (78.7, 67.1)
- moved REF** 0.76 mm to (82.5, 66.3)
Changed lines of the file:
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@@
 	(footprint "Connector_Wire:SolderWire-0.5sqmm_1x01_D0.9mm_OD2.3mm"
 		(layer "F.Cu")
-		(at 82.55 65.532)
+		(at 82.55 66.294)
 		(descr "Soldered wire connection, for a single 0.5 mm² wire, reinforced insulation, conductor diameter 0.9mm, outer diameter 2.3mm, size source Multi-Contact FLEXI-xV 0.5 (https://ec.staubli.com/AcroFiles/Catalogues/TM_Cab-Main-11014119_(en)_hi.pdf), bend radius 3 times outer diameter, generated with kicad-footprint-generator")
 		(tags "connector wire 0.5sqmm")
@@
 	(footprint "Connector_Wire:SolderWire-0.5sqmm_1x01_D0.9mm_OD2.3mm"
 		(layer "F.Cu")
-		(at 79.502 67.31)
+		(at 78.74 67.056)
 		(descr "Soldered wire connection, for a single 0.5 mm² wire, reinforced insulation, conductor diameter 0.9mm, outer diameter 2.3mm, size source Multi-Contact FLEXI-xV 0.5 (https://ec.staubli.com/AcroFiles/Catalogues/TM_Cab-Main-11014119_(en)_hi.pdf), bend radius 3 times outer diameter, generated with kicad-footprint-generator")
 		(tags "connector wire 0.5sqmm")
@@
 	)
 	(segment
-		(start 85.62 73.12)
-		(end 80.12 67.62)
+		(start 84.804 73.12)
+		(end 78.74 67.056)
 		(width 0.5)
 		(layer "F.Cu")
@@
 	)
 	(segment
+		(start 85.62 73.12)
+		(end 84.804 73.12)
+		(width 0.5)
+		(layer "F.Cu")
+		(net 12)
+	)
+	(segment
 		(start 89.12 83.62)
 		(end 75.62 83.62)
@@
 	)
 	(segment
-		(start 79.502 67.002)
-		(end 79.502 61.252)
+		(start 78.18 59.93)
+		(end 69.205 59.93)
 		(width 0.5)
 		(layer "B.Cu")
@@
 	)
 	(segment
+		(start 78.74 67.056)
+		(end 78.74 60.49)
+		(width 0.5)
+		(layer "B.Cu")
+		(net 12)
+	)
+	(segment
 		(start 91.62 81.12)
 		(end 89.12 83.62)
@@
 	)
 	(segment
-		(start 79.502 61.252)
+		(start 78.74 60.49)
 		(end 78.18 59.93)
-		(width 0.5)
-		(layer "B.Cu")
-		(net 12)
-	)
-	(segment
-		(start 80.12 67.62)
-		(end 79.502 67.002)
 		(width 0.5)
 		(layer "B.Cu")
@@
 		(width 0.5)
 		(layer "B.Cu")
-		(net 12)
-	)
-	(segment
-		(start 78.18 59.93)
-		(end 69.205 59.93)
-		(width 0.5)
-		(layer "B.Cu")
